File: solar_converter/solar_converter.kicad_sch (KiCad schematic)
At the start: 35 parts, among them J1 Conn_01x02_Pin, Q1 IRLB8721PBF, Q2 IRLB8721PBF, Q3 IRLB8721PBF, Q4 IRLB8721PBF, Q5 IRLB8721PBF, Q6 IRLB8721PBF, Q7 IRLB8721PBF, U1 LM324, U2 ACS712xLCTR-05B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

Commit message: add some values to schematic
Parts:
- removed D1: SB140, Diode_THT:D_DO-41_SOD81_P10.16mm_Horizontal, symbol Diode:SB140
- removed Q1: IRLB8721PBF, Package_TO_SOT_THT:TO-220-3_Vertical, symbol Transistor_FET:IRLB8721PBF
- added C4: 100u, symbol Device:C_Polarized_US
- added L3: 320m, symbol Device:L
- added R17, R19, R20: 100k, symbol Device:R_US
- added R18: 330k, symbol Device:R_US
- C1, C2: value C_Polarized_US -> 470u
- C3: value C_Polarized_US -> 100u
- L1, L2: value L -> 320m
- R1: value R_US -> R_load
- R14, R16, R4, R5: value R_US -> 100
- R15, R3: value R_US -> 10k
- R2: value R_US -> 1k
Connections:
- net GND: now also R18.2, R20.2
- net V+: now also L3.1
- net V_pwm1: now also U3.13 (PH1)
- net V_pwm2: now also U3.12 (PH0)
- net at C1.2, C2.2, C3.2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: now also L1.1
- net V_fb_1_stepdown: now reaches U1.1
- net V_fb_1_stepdown: now also U1.2 (-), U3.55 (PC2), U3.57 (PC4)
- net at U1.3 (+): now also R17.2, R18.1
- net V_fb_2: now reaches C3.1, L2.2, R2.1
- net V_fb_2: now also R19.1
- net V_fb_1: now reaches C1.1, D2.1 (K), R1.1
- net V_fb_1: now also R17.1
- net at D2.2 (A), L1.2: now also C4.2; no longer Q2.2 (D)
- net at U1.5 (+): now also R19.2, R20.1
- net V_fb_2_stepdown: now reaches U1.6 (-)
- net V_fb_2_stepdown: now also U1.7, U3.54 (PC1)
- net V_fault: now reaches U3.22 (PB3)
- net ADC_flag: now reaches U3.23 (PB4)
- net MPPT_en: now reaches U3.24 (PB5)
- net MPPT_on_sw: now reaches U3.25 (PB6)
- net MPPT_flag: now reaches U3.26 (PB7)
- new net: C4.1, L3.2, Q2.2 (D)
Other:
- note added: "Not pictured: connections with the ATMega2560 on the Arduino Mega PCB"
- moved on the sheet: Q2
